File: turbo_jumper.brd (EAGLE design)
At the start: 72.4 x 50.5 mm, 8 parts, among them X1 E74, X2 P-remote

Commit message: up
Parts:
- added K1: 351, relay:351
Connections:
- removed net ACCEL-: X1.11
- net 24+_REMOTE_PRI: now also K1.1, LED3.A, X2.14; no longer X2.23
- net ACCEL+: now also K1.S2
- net N$1: now also K1.P2, X2.15; no longer LED3.A, X2.14
- net NORM-: now also X1.11
- net START-: now also K1.16
Routing:
- net ACCEL+: track 0.00 -> 32.6 mm
- net 24+_REMOTE_PRI: track 68.3 -> 82.4 mm
- net START-: track 43.1 -> 54.4 mm
- net N$1: track 36.2 -> 26.6 mm
- net ALARM+: track 65.4 -> 59.5 mm
- net NORM-: track 42.6 -> 45.4 mm
- net ALARM-: track 55.0 -> 55.7 mm

Commit message: up
Parts:
- removed K1: 351, relay:351
- added K2: G2R2, relay:G2R2
- added SV1: AUX-SW, con-lstb:MA03-1
- moved X2 7.62 mm to (104.1, 57.1)
Connections:
- new net N$5: K2.O1, SV1.2
- new net N$6: K2.S1, SV1.1
- new net NOT_NORM: K2.P2, X2.15
- net 24+_REMOTE_PRI: no longer K1.1
- net ACCEL+: now also K2.S2; no longer K1.S2
- net GND: now also K2.2
- net N$1: now also K2.P1, SV1.3; no longer K1.P2, X2.15
- net START-: now also K2.1; no longer K1.16
Routing:
- net NORM+: track 55.1 -> 105.4 mm
- net GND: track 4.21 -> 39.8 mm, vias 3 -> 0
- net 24+_REMOTE_PRI: track 82.4 -> 110.3 mm
- net ACCEL+: track 32.6 -> 59.1 mm
- net START-: track 54.4 -> 75.6 mm
- net ALARM-: track 55.7 -> 76.3 mm
- net NOT_NORM: track 0.00 -> 20.2 mm
- net ALARM+: track 59.5 -> 78.0 mm
- net N$1: track 26.6 -> 8.35 mm
- net N$6: track 0.00 -> 14.1 mm
- net NORM-: track 45.4 -> 58.7 mm, vias 0 -> 1
- net N$5: track 0.00 -> 12.9 mm
- net ERROR: track 14.4 -> 22.0 mm
- net SPEED: track 12.7 -> 20.3 mm

Commit message: up
Parts:
- removed K2: G2R2, relay:G2R2
- added K1: G6K-2P, relay:G6K-2P
- moved SV1 14.2 mm to (90.2, 59.7)
Connections:
- removed net N$1: K2.P1, SV1.3
- removed net N$5: K2.O1, SV1.2
- removed net N$6: K2.S1, SV1.1
- new net R-COM: K1.3, SV1.3
- new net R-NC: K1.2, SV1.2
- new net R-NO: K1.4, SV1.1
- net ACCEL+: now also K1.5; no longer K2.S2
- net GND: now also K1.8; no longer K2.2
- net NOT_NORM: now also K1.6; no longer K2.P2
- net START-: now also K1.1; no longer K2.1
Routing:
- net 24+_REMOTE_PRI: track 110.3 -> 65.2 mm
- net ACCEL+: track 59.1 -> 30.6 mm, vias 0 -> 1
- net R-NC: track 0.00 -> 15.8 mm
- net N$6: track 14.1 -> 0.00 mm
- net START-: track 75.6 -> 88.7 mm
- net N$5: track 12.9 -> 0.00 mm
- net R-COM: track 0.00 -> 11.5 mm
- net R-NO: track 0.00 -> 9.72 mm
- net NORM-: track 58.7 -> 68.3 mm, vias 1 -> 0
- net N$1: track 8.35 -> 0.00 mm
- net NOT_NORM: track 20.2 -> 27.9 mm
- net GND: track 39.8 -> 35.3 mm
Other:
- board text added: "V1.0 E74 to TM700 connector adapter"

Commit message: up
Parts:
- removed X2: P-remote, con-subd:HDF26V
- added DCU: DCU, con-lstb:MA08-1
- added J1: 10090926-P264XLF, 10090926-P264XLF:10090926P264XLF
- added SV2: ANALOG OUT, con-lstb:MA03-1
- added TP1, TP2, TP3, TP4, TP5, TP6, TP7, TP8: TPSQTP13R, testpad:TP13R
- moved SV1 22.9 mm to (67.3, 58.4), flipped to the bottom
- moved R3 8.98 mm to (67.3, 73.7), turned to 0 degrees
- moved LED3 6.48 mm to (74.9, 73.7), flipped to the bottom, turned to 90 degrees
- moved LED1 6.35 mm to (74.9, 47.0), flipped to the bottom
- moved LED2 6.35 mm to (74.9, 40.6), flipped to the bottom
- moved R1 6.35 mm to (67.3, 47.0)
- moved R2 6.35 mm to (67.3, 40.6)
- moved K1 4.02 mm to (81.3, 58.4)
- turned X1 to 270 degrees
Connections:
- new net AO1: J1.12, SV2.1
- new net D+: DCU.1, J1.24
- new net D-: DCU.2, J1.25
- new net REMOTE_ACTIVE: J1.23, LED3.A, TP5.TP
- net 24+_REMOTE_PRI: now also DCU.7, J1.1, J1.14, TP3.TP; no longer LED3.A, X2.1, X2.14
- net ALARM+: now also J1.19; no longer X2.19
- net ALARM-: now also J1.20; no longer X2.20
- net ERROR: now also J1.9; no longer X2.9
- net GND: now also DCU.8, J1.26, SV2.3, TP1.TP; no longer X2.26
- net NORM+: now also J1.17, TP6.TP; no longer X2.17
- net NORM-: now also J1.16, TP7.TP; no longer X2.16
- net NOT_NORM: now also J1.15, TP8.TP; no longer X2.15
- net SPEED: now also J1.8; no longer X2.8
- net START-: now also J1.3, J1.4, TP2.TP, TP4.TP; no longer X2.3, X2.4
Routing:
- net REMOTE_ACTIVE: track 0.00 -> 79.7 mm
- net AO1: track 0.00 -> 36.4 mm, vias 0 -> 1
- net NORM-: track 68.3 -> 103.5 mm, vias 0 -> 3
- net NOT_NORM: track 27.9 -> 58.7 mm, vias 0 -> 2
- net D+: track 0.00 -> 30.6 mm
- net 24+_REMOTE_PRI: track 65.2 -> 94.6 mm, vias 0 -> 1
- net D-: track 0.00 -> 28.2 mm
- net START-: track 88.7 -> 65.8 mm
- net ERROR: track 22.0 -> 43.1 mm, vias 0 -> 2
- net SPEED: track 20.3 -> 40.5 mm, vias 0 -> 2
- net ALARM+: track 78.0 -> 63.6 mm
- net R-NO: track 9.72 -> 21.2 mm
- net GND: track 35.3 -> 26.7 mm, vias 0 -> 1
- net R-COM: track 11.5 -> 17.3 mm
- net ALARM-: track 76.3 -> 81.5 mm
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
Commit message: up
Routing:
- net ALARM+: track 63.6 -> 77.4 mm
- net NORM+: track 105.6 -> 117.3 mm
- net ALARM-: track 81.5 -> 73.2 mm
- net START-: track 65.8 -> 72.7 mm
- net REMOTE_ACTIVE: track 79.7 -> 85.7 mm, vias 0 -> 1
- net ERROR: track 43.1 -> 48.0 mm, vias 2 -> 3
- net NORM-: track 103.5 -> 105.9 mm
- net D-: track 28.2 -> 26.4 mm
- net AO1: track 36.4 -> 37.8 mm
- net NOT_NORM: track 58.7 -> 60.1 mm, vias 2 -> 3
- net D+: track 30.6 -> 31.2 mm

Commit message: up
Parts:
- added K2: G6K-2P-Y, relay:G6K-2P-Y
- K1: value G6K-2P -> G6K-2P-Y; device relay:G6K-2P -> relay:G6K-2P-Y
- moved K1 6.35 mm to (74.9, 58.4)
Connections:
- net R-NO renamed N$5
- removed net R-COM: K1.3, SV1.3
- removed net R-NC: K1.2, SV1.2
- new net DECEL_STOP: K1.2, K2.1, SV1.2
- net DECEL+: now also K2.6
- net DECEL-: now also K2.5
- net GND: now also K2.8
- net SPEED: now also K1.3, SV1.3
Routing:
- net GND: track 26.6 -> 86.1 mm, vias 1 -> 0
- net DECEL-: track 0.00 -> 28.4 mm, vias 0 -> 1
- net DECEL+: track 0.00 -> 23.4 mm
- net DECEL_STOP: track 0.00 -> 18.2 mm
- net R-COM: track 17.4 -> 0.00 mm
- net R-NC: track 15.0 -> 0.00 mm
- net SPEED: track 40.4 -> 53.2 mm, vias 2 -> 1
- net ALARM+: track 77.4 -> 66.2 mm
- net ALARM-: track 73.2 -> 81.8 mm
- net REMOTE_ACTIVE: track 85.7 -> 79.4 mm, vias 1 -> 2
- net N$5: track 21.2 -> 25.6 mm
- net NOT_NORM: track 60.1 -> 63.8 mm, vias 3 -> 2
- net N$4: track 8.08 -> 9.65 mm
- net 24+_REMOTE_PRI: track 95.0 -> 93.7 mm
- net NORM+: track 117.3 -> 118.6 mm
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
Commit message: up
Parts:
- removed DCU: DCU, con-lstb:MA08-1
- removed LED1: speed, led:CHIPLED_1206
- removed LED2: error, led:CHIPLED_1206
- removed LED3: in remote, led:CHIPLED_1206
- removed R1, R2, R3: 10k, rcl:M1206
- removed SV1: AUX-SW, con-lstb:MA03-1
- removed SV2: ANALOG OUT, con-lstb:MA03-1
- removed TP1, TP2, TP3, TP4, TP5, TP6, TP7, TP8: TPSQTP13R, testpad:TP13R
- moved K1 6.35 mm to (74.9, 52.1)
- moved K2 5.24 mm to (74.9, 66.0)
Connections:
- removed net 24+_REMOTE_PRI: DCU.7, J1.1, J1.14, TP3.TP, X1.1
- removed net ACCEL+: K1.5, X1.3
- removed net AO1: J1.12, SV2.1
- removed net D+: DCU.1, J1.24
- removed net D-: DCU.2, J1.25
- removed net DECEL+: K2.6, X1.5
- removed net DECEL-: K2.5, X1.13
- removed net DECEL_STOP: K1.2, K2.1, SV1.2
- removed net GND: DCU.8, J1.26, K1.8, K2.8, R1.1, R2.1, R3.1, SV2.3, TP1.TP
- removed net N$2: LED3.C, R3.2
- removed net N$3: LED1.C, R1.2
- removed net N$4: LED2.C, R2.2
- removed net N$5: K1.4, SV1.1
- removed net NOT_NORM: J1.15, K1.6, TP8.TP
- removed net REMOTE_ACTIVE: J1.23, LED3.A, TP5.TP
- new net P_GND: J1.26, K1.8, K2.8
- new net START+: J1.1, J1.14, J1.2, J1.4, X1.1
- net ALARM+: now also K1.3, X1.8; no longer J1.19, X1.6
- net ALARM-: now also K1.2; no longer J1.20
- net ERROR: now also K1.1; no longer LED2.A
- net NORM+: now also K2.3; no longer J1.17, TP6.TP
- net NORM-: now also K2.4; no longer J1.16, TP7.TP, X1.11
- net SPEED: now also K2.1; no longer K1.3, LED1.A, SV1.3
- net START-: no longer J1.4, K1.1, TP2.TP, TP4.TP
Routing:
- net 24+_REMOTE_PRI: track 93.7 -> 0.00 mm, vias 1 -> 0
- net NORM+: track 118.6 -> 27.0 mm, vias 1 -> 0
- net GND: track 86.1 -> 0.00 mm
- net REMOTE_ACTIVE: track 79.4 -> 0.00 mm, vias 2 -> 0
- net NORM-: track 105.5 -> 32.3 mm, vias 3 -> 0
- net NOT_NORM: track 63.8 -> 0.00 mm, vias 2 -> 0
- net START+: track 0.00 -> 60.0 mm
- net P_GND: track 0.00 -> 51.7 mm
- net ALARM-: track 81.8 -> 36.9 mm
- net AO1: track 36.7 -> 0.00 mm, vias 1 -> 0
- net ACCEL+: track 33.9 -> 0.00 mm
- net D+: track 30.3 -> 0.00 mm
- net DECEL-: track 28.4 -> 0.00 mm, vias 1 -> 0
- net D-: track 26.4 -> 0.00 mm
- net N$5: track 25.6 -> 0.00 mm
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Other:
- board text added: "V1.1 V E74 to TM700 connector adapter"
- board text removed: "V1.0 E74 to TM700 connector adapter"
