File: turbo_jumper.sch (EAGLE design)
At the start: 8 parts, among them X1 E74, X2 P-remote

Commit message: up
Parts:
- added K1: 351, relay:351
Connections:
- removed net ACCEL-: X1.11
- net 24+_REMOTE_PRI: now also K11.1, LED3.A, X2.14; no longer X2.23
- net ACCEL+: now also K13.S
- net N$1: now also K13.P, X2.15; no longer LED3.A, X2.14
- net NORM-: now also X1.11
- net START-: now also K11.2
Changed lines of the file:
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@@
 <part name="R3" library="rcl" library_urn="urn:adsk.eagle:library:334" deviceset="R-US_" device="M1206" package3d_urn="urn:adsk.eagle:package:23566/2" value="10k"/>
 <part name="GND4" library="supply1" library_urn="urn:adsk.eagle:library:371" deviceset="GND" device=""/>
+<part name="K1" library="relay" library_urn="urn:adsk.eagle:library:339" deviceset="351" device="" package3d_urn="urn:adsk.eagle:package:24300/1"/>
 </parts>
 <sheets>
 <sheet>
 <plain>
-<text x="106.68" y="53.34" size="1.778" layer="91">remote active
+<text x="66.04" y="55.88" size="1.778" layer="91">remote active
 jumper to pin 1</text>
 <text x="27.94" y="73.66" size="1.778" layer="91">relay on during turbo start</text>
@@
 <attribute name="VALUE" x="40.64" y="45.72" size="1.778" layer="96"/>
 </instance>
+<instance part="K1" gate="1" x="33.02" y="96.52" smashed="yes">
+<attribute name="VALUE" x="34.29" y="99.441" size="1.778" layer="96"/>
+<attribute name="PART" x="34.29" y="101.6" size="1.778" layer="95"/>
+</instance>
+<instance part="K1" gate="2" x="50.8" y="93.98" smashed="yes">
+<attribute name="PART" x="53.34" y="93.98" size="1.778" layer="95"/>
+</instance>
+<instance part="K1" gate="3" x="50.8" y="78.74" smashed="yes">
+<attribute name="PART" x="53.34" y="78.74" size="1.778" layer="95"/>
+</instance>
 </instances>
 <busses>
@@
 </segment>
 <segment>
-<wire x1="106.68" y1="55.88" x2="101.6" y2="55.88" width="0.1524" layer="91"/>
-<pinref part="X2" gate="G$1" pin="23"/>
-<label x="101.6" y="58.42" size="1.778" layer="95"/>
-<junction x="96.52" y="55.88"/>
-<junction x="106.68" y="55.88"/>
-<wire x1="101.6" y1="55.88" x2="96.52" y2="55.88" width="0.1524" layer="91"/>
-<wire x1="101.6" y1="55.88" x2="101.6" y2="63.5" width="0.1524" layer="91"/>
-<junction x="101.6" y="55.88"/>
-<wire x1="101.6" y1="63.5" x2="121.92" y2="63.5" width="0.1524" layer="91"/>
-<wire x1="121.92" y1="63.5" x2="121.92" y2="88.9" width="0.1524" layer="91"/>
-<wire x1="121.92" y1="88.9" x2="76.2" y2="88.9" width="0.1524" layer="91"/>
-<wire x1="81.28" y1="76.2" x2="76.2" y2="76.2" width="0.1524" layer="91"/>
 <pinref part="X2" gate="G$1" pin="1"/>
 <label x="58.42" y="78.74" size="1.778" layer="95"/>
 <junction x="81.28" y="76.2"/>
 <junction x="71.12" y="76.2"/>
-<wire x1="76.2" y1="76.2" x2="71.12" y2="76.2" width="0.1524" layer="91"/>
-<wire x1="76.2" y1="88.9" x2="76.2" y2="76.2" width="0.1524" layer="91"/>
-<junction x="76.2" y="76.2"/>
+<wire x1="81.28" y1="76.2" x2="73.66" y2="76.2" width="0.1524" layer="91"/>
+<wire x1="73.66" y1="76.2" x2="71.12" y2="76.2" width="0.1524" layer="91"/>
+<wire x1="73.66" y1="76.2" x2="73.66" y2="73.66" width="0.1524" layer="91"/>
+<junction x="73.66" y="76.2"/>
+<wire x1="73.66" y1="73.66" x2="60.96" y2="73.66" width="0.1524" layer="91"/>
+<pinref part="X2" gate="G$1" pin="14"/>
+<wire x1="81.28" y1="58.42" x2="60.96" y2="58.42" width="0.1524" layer="91"/>
+<wire x1="60.96" y1="58.42" x2="60.96" y2="50.8" width="0.1524" layer="91"/>
+<pinref part="LED3" gate="G$1" pin="A"/>
+<junction x="60.96" y="50.8"/>
+<junction x="81.28" y="58.42"/>
+<wire x1="60.96" y1="73.66" x2="60.96" y2="58.42" width="0.1524" layer="91"/>
+<junction x="60.96" y="58.42"/>
+</segment>
+<segment>
+<wire x1="33.02" y1="101.6" x2="22.86" y2="101.6" width="0.1524" layer="91"/>
+<pinref part="K1" gate="1" pin="1"/>
+<label x="25.4" y="104.14" size="1.778" layer="95"/>
+<junction x="33.02" y="101.6"/>
+<junction x="22.86" y="101.6"/>
 </segment>
 </net>
@@
 <junction x="71.12" y="60.96"/>
 </segment>
+<segment>
+<wire x1="22.86" y1="91.44" x2="33.02" y2="91.44" width="0.1524" layer="91"/>
+<pinref part="K1" gate="1" pin="2"/>
+<label x="27.94" y="88.9" size="1.778" layer="95"/>
+<junction x="33.02" y="91.44"/>
+<junction x="22.86" y="91.44"/>
+</segment>
 </net>
 <net name="ALARM-" class="0">
@@
 <junction x="5.08" y="63.5"/>
 </segment>
-</net>
-<net name="ACCEL-" class="0">
-<segment>
-<pinref part="X1" gate="-1" pin="11"/>
-<wire x1="30.48" y1="63.5" x2="40.64" y2="63.5" width="0.1524" layer="91"/>
-<label x="40.64" y="63.5" size="1.778" layer="95"/>
-<junction x="30.48" y="63.5"/>
-<junction x="40.64" y="63.5"/>
+<segment>
+<wire x1="45.72" y1="83.82" x2="35.56" y2="83.82" width="0.1524" layer="91"/>
+<pinref part="K1" gate="3" pin="S"/>
+<label x="38.1" y="81.28" size="1.778" layer="95"/>
+<junction x="45.72" y="83.82"/>
+<junction x="35.56" y="83.82"/>
 </segment>
 </net>
@@
 <segment>
 <pinref part="X1" gate="-1" pin="12"/>
-<wire x1="30.48" y1="60.96" x2="40.64" y2="60.96" width="0.1524" layer="91"/>
+<wire x1="30.48" y1="60.96" x2="38.1" y2="60.96" width="0.1524" layer="91"/>
 <label x="40.64" y="60.96" size="1.778" layer="95"/>
 <junction x="30.48" y="60.96"/>
 <junction x="40.64" y="60.96"/>
+<pinref part="X1" gate="-1" pin="11"/>
+<wire x1="38.1" y1="60.96" x2="40.64" y2="60.96" width="0.1524" layer="91"/>
+<wire x1="30.48" y1="63.5" x2="38.1" y2="63.5" width="0.1524" layer="91"/>
+<label x="40.64" y="63.5" size="1.778" layer="95"/>
+<junction x="30.48" y="63.5"/>
+<junction x="40.64" y="63.5"/>
+<wire x1="38.1" y1="63.5" x2="40.64" y2="63.5" width="0.1524" layer="91"/>
+<wire x1="38.1" y1="60.96" x2="38.1" y2="63.5" width="0.1524" layer="91"/>
+<junction x="38.1" y="60.96"/>
+<junction x="38.1" y="63.5"/>
 </segment>
 <segment>
@@
 </segment>
 </net>
-<net name="N$1" class="0">
-<segment>
-<pinref part="X2" gate="G$1" pin="14"/>
-<wire x1="81.28" y1="58.42" x2="60.96" y2="58.42" width="0.1524" layer="91"/>
-<wire x1="60.96" y1="58.42" x2="60.96" y2="50.8" width="0.1524" layer="91"/>
-<pinref part="LED3" gate="G$1" pin="A"/>
-<junction x="60.96" y="50.8"/>
-<junction x="81.28" y="58.42"/>
-</segment>
-</net>
 <net name="N$2" class="0">
 <segment>
@@
 </segment>
 </net>
+<net name="N$1" class="0">
+<segment>
+<pinref part="K1" gate="3" pin="P"/>
+<wire x1="50.8" y1="76.2" x2="58.42" y2="76.2" width="0.1524" layer="91"/>
+<wire x1="58.42" y1="76.2" x2="58.42" y2="55.88" width="0.1524" layer="91"/>
+<pinref part="X2" gate="G$1" pin="15"/>
+<wire x1="81.28" y1="53.34" x2="63.5" y2="53.34" width="0.1524" layer="91"/>
+<wire x1="63.5" y1="53.34" x2="63.5" y2="55.88" width="0.1524" layer="91"/>
+<wire x1="63.5" y1="55.88" x2="58.42" y2="55.88" width="0.1524" layer="91"/>
+<junction x="50.8" y="76.2"/>
+<junction x="81.28" y="53.34"/>
+</segment>
+</net>

Commit message: up
Parts:
- removed K1: 351, relay:351
- added K2: G2R2, relay:G2R2
- added SV1: AUX-SW, con-lstb:MA03-1
Connections:
- new net N$5: K22.O, SV1.2
- new net N$6: K22.S, SV1.1
- new net NOT_NORM: K23.P, X2.15
- net 24+_REMOTE_PRI: no longer K11.1
- net ACCEL+: now also K23.S; no longer K13.S
- net GND: now also K21.2
- net N$1: now also K22.P, SV1.3; no longer K13.P, X2.15
- net START-: now also K21.1; no longer K11.2
Changed lines of the file:
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@@
 <part name="R3" library="rcl" library_urn="urn:adsk.eagle:library:334" deviceset="R-US_" device="M1206" package3d_urn="urn:adsk.eagle:package:23566/2" value="10k"/>
 <part name="GND4" library="supply1" library_urn="urn:adsk.eagle:library:371" deviceset="GND" device=""/>
-<part name="K1" library="relay" library_urn="urn:adsk.eagle:library:339" deviceset="351" device="" package3d_urn="urn:adsk.eagle:package:24300/1"/>
+<part name="K2" library="relay" library_urn="urn:adsk.eagle:library:339" deviceset="G2R2" device="" package3d_urn="urn:adsk.eagle:package:24328/1"/>
+<part name="GND6" library="supply1" library_urn="urn:adsk.eagle:library:371" deviceset="GND" device=""/>
+<part name="SV1" library="con-lstb" library_urn="urn:adsk.eagle:library:162" deviceset="MA03-1" device="" package3d_urn="urn:adsk.eagle:package:8339/1" value="AUX-SW"/>
 </parts>
 <sheets>
@@
 <attribute name="VALUE" x="40.64" y="45.72" size="1.778" layer="96"/>
 </instance>
-<instance part="K1" gate="1" x="33.02" y="96.52" smashed="yes">
-<attribute name="VALUE" x="34.29" y="99.441" size="1.778" layer="96"/>
-<attribute name="PART" x="34.29" y="101.6" size="1.778" layer="95"/>
-</instance>
-<instance part="K1" gate="2" x="50.8" y="93.98" smashed="yes">
-<attribute name="PART" x="53.34" y="93.98" size="1.778" layer="95"/>
-</instance>
-<instance part="K1" gate="3" x="50.8" y="78.74" smashed="yes">
-<attribute name="PART" x="53.34" y="78.74" size="1.778" layer="95"/>
+<instance part="K2" gate="1" x="27.94" y="93.98" smashed="yes">
+<attribute name="VALUE" x="29.21" y="96.901" size="1.778" layer="96"/>
+<attribute name="PART" x="29.21" y="99.06" size="1.778" layer="95"/>
+</instance>
+<instance part="K2" gate="2" x="48.26" y="101.6" smashed="yes">
+<attribute name="PART" x="50.8" y="101.6" size="1.778" layer="95"/>
+</instance>
+<instance part="K2" gate="3" x="48.26" y="86.36" smashed="yes">
+<attribute name="PART" x="50.8" y="86.36" size="1.778" layer="95"/>
+</instance>
+<instance part="GND6" gate="1" x="27.94" y="86.36" smashed="yes">
+<attribute name="VALUE" x="25.4" y="83.82" size="1.778" layer="96"/>
+</instance>
+<instance part="SV1" gate="G$1" x="78.74" y="101.6" smashed="yes" rot="R180">
+<attribute name="VALUE" x="80.01" y="109.22" size="1.778" layer="96" rot="R180"/>
+<attribute name="NAME" x="80.01" y="95.758" size="1.778" layer="95" rot="R180"/>
 </instance>
 </instances>
@@
 <junction x="60.96" y="58.42"/>
 </segment>
-<segment>
-<wire x1="33.02" y1="101.6" x2="22.86" y2="101.6" width="0.1524" layer="91"/>
-<pinref part="K1" gate="1" pin="1"/>
-<label x="25.4" y="104.14" size="1.778" layer="95"/>
-<junction x="33.02" y="101.6"/>
-<junction x="22.86" y="101.6"/>
-</segment>
 </net>
 <net name="START-" class="0">
@@
 </segment>
 <segment>
-<wire x1="22.86" y1="91.44" x2="33.02" y2="91.44" width="0.1524" layer="91"/>
-<pinref part="K1" gate="1" pin="2"/>
-<label x="27.94" y="88.9" size="1.778" layer="95"/>
-<junction x="33.02" y="91.44"/>
-<junction x="22.86" y="91.44"/>
+<wire x1="20.32" y1="99.06" x2="27.94" y2="99.06" width="0.1524" layer="91"/>
+<pinref part="K2" gate="1" pin="1"/>
+<label x="20.32" y="101.6" size="1.778" layer="95"/>
+<junction x="20.32" y="99.06"/>
+<junction x="27.94" y="99.06"/>
 </segment>
 </net>
@@
 </segment>
 <segment>
-<wire x1="45.72" y1="83.82" x2="35.56" y2="83.82" width="0.1524" layer="91"/>
-<pinref part="K1" gate="3" pin="S"/>
-<label x="38.1" y="81.28" size="1.778" layer="95"/>
-<junction x="45.72" y="83.82"/>
-<junction x="35.56" y="83.82"/>
+<wire x1="43.18" y1="91.44" x2="43.18" y2="93.98" width="0.1524" layer="91"/>
+<pinref part="K2" gate="3" pin="S"/>
+<label x="45.72" y="93.98" size="1.778" layer="95"/>
+<junction x="43.18" y="91.44"/>
+<junction x="43.18" y="93.98"/>
 </segment>
 </net>
@@
 <junction x="43.18" y="50.8"/>
 </segment>
+<segment>
+<pinref part="K2" gate="1" pin="2"/>
+<pinref part="GND6" gate="1" pin="GND"/>
+<junction x="27.94" y="88.9"/>
+</segment>
 </net>
 <net name="ERROR" class="0">
@@
 </segment>
 </net>
-<net name="N$1" class="0">
-<segment>
-<pinref part="K1" gate="3" pin="P"/>
-<wire x1="50.8" y1="76.2" x2="58.42" y2="76.2" width="0.1524" layer="91"/>
+<net name="NOT_NORM" class="0">
+<segment>
 <wire x1="58.42" y1="76.2" x2="58.42" y2="55.88" width="0.1524" layer="91"/>
 <pinref part="X2" gate="G$1" pin="15"/>
@@
 <wire x1="63.5" y1="53.34" x2="63.5" y2="55.88" width="0.1524" layer="91"/>
 <wire x1="63.5" y1="55.88" x2="58.42" y2="55.88" width="0.1524" layer="91"/>
-<junction x="50.8" y="76.2"/>
 <junction x="81.28" y="53.34"/>
-</segment>
-</net>
+<label x="53.34" y="76.2" size="1.778" layer="95"/>
+<junction x="58.42" y="76.2"/>
+</segment>
+<segment>
+<wire x1="48.26" y1="83.82" x2="55.88" y2="83.82" width="0.1524" layer="91"/>
+<pinref part="K2" gate="3" pin="P"/>
+<label x="58.42" y="83.82" size="1.778" layer="95"/>
+<junction x="48.26" y="83.82"/>
+<junction x="55.88" y="83.82"/>
+</segment>
+</net>
+<net name="N$1" class="0">
+<segment>
+<pinref part="K2" gate="2" pin="P"/>
+<pinref part="SV1" gate="G$1" pin="3"/>
+<wire x1="48.26" y1="99.06" x2="71.12" y2="99.06" width="0.1524" layer="91"/>
+<junction x="48.26" y="99.06"/>
+<junction x="71.12" y="99.06"/>
+</segment>
+</net>
+<net name="N$5" class="0">
+<segment>
+<pinref part="K2" gate="2" pin="O"/>
+<wire x1="53.34" y1="106.68" x2="55.88" y2="106.68" width="0.1524" layer="91"/>
+<wire x1="55.88" y1="106.68" x2="55.88" y2="101.6" width="0.1524" layer="91"/>
+<pinref part="SV1" gate="G$1" pin="2"/>
+<wire x1="55.88" y1="101.6" x2="71.12" y2="101.6" width="0.1524" layer="91"/>
+<junction x="53.34" y="106.68"/>
+<junction x="71.12" y="101.6"/>
+</segment>
+</net>
+<net name="N$6" class="0">
+<segment>
+<pinref part="SV1" gate="G$1" pin="1"/>
+<wire x1="71.12" y1="104.14" x2="71.12" y2="109.22" width="0.1524" layer="91"/>
+<wire x1="71.12" y1="109.22" x2="43.18" y2="109.22" width="0.1524" layer="91"/>
+<pinref part="K2" gate="2" pin="S"/>
+<wire x1="43.18" y1="109.22" x2="43.18" y2="106.68" width="0.1524" layer="91"/>
+<junction x="43.18" y="106.68"/>
+<junction x="71.12" y="104.14"/>
+</segment>
+</net>

Commit message: up
Parts:
- removed K2: G2R2, relay:G2R2
- added K1: G6K-2P, relay:G6K-2P
Connections:
- removed net N$1: K22.P, SV1.3
- removed net N$5: K22.O, SV1.2
- removed net N$6: K22.S, SV1.1
- new net R-COM: K12.P, SV1.3
- new net R-NC: K12.O, SV1.2
- new net R-NO: K12.S, SV1.1
- net ACCEL+: now also K13.S; no longer K23.S
- net GND: now also K11.-; no longer K21.2
- net NOT_NORM: now also K13.P; no longer K23.P
- net START-: now also K11.+; no longer K21.1
Other:
- moved on the sheet: SV1
Changed lines of the file:
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@@
 <part name="R3" library="rcl" library_urn="urn:adsk.eagle:library:334" deviceset="R-US_" device="M1206" package3d_urn="urn:adsk.eagle:package:23566/2" value="10k"/>
 <part name="GND4" library="supply1" library_urn="urn:adsk.eagle:library:371" deviceset="GND" device=""/>
-<part name="K2" library="relay" library_urn="urn:adsk.eagle:library:339" deviceset="G2R2" device="" package3d_urn="urn:adsk.eagle:package:24328/1"/>
-<part name="GND6" library="supply1" library_urn="urn:adsk.eagle:library:371" deviceset="GND" device=""/>
 <part name="SV1" library="con-lstb" library_urn="urn:adsk.eagle:library:162" deviceset="MA03-1" device="" package3d_urn="urn:adsk.eagle:package:8339/1" value="AUX-SW"/>
+<part name="K1" library="relay" library_urn="urn:adsk.eagle:library:339" deviceset="G6K" device="-2P" package3d_urn="urn:adsk.eagle:package:24346/1"/>
+<part name="GND5" library="supply1" library_urn="urn:adsk.eagle:library:371" deviceset="GND" device=""/>
 </parts>
 <sheets>
@@
 <attribute name="VALUE" x="40.64" y="45.72" size="1.778" layer="96"/>
 </instance>
-<instance part="K2" gate="1" x="27.94" y="93.98" smashed="yes">
-<attribute name="VALUE" x="29.21" y="96.901" size="1.778" layer="96"/>
-<attribute name="PART" x="29.21" y="99.06" size="1.778" layer="95"/>
-</instance>
-<instance part="K2" gate="2" x="48.26" y="101.6" smashed="yes">
-<attribute name="PART" x="50.8" y="101.6" size="1.778" layer="95"/>
-</instance>
-<instance part="K2" gate="3" x="48.26" y="86.36" smashed="yes">
-<attribute name="PART" x="50.8" y="86.36" size="1.778" layer="95"/>
-</instance>
-<instance part="GND6" gate="1" x="27.94" y="86.36" smashed="yes">
-<attribute name="VALUE" x="25.4" y="83.82" size="1.778" layer="96"/>
-</instance>
-<instance part="SV1" gate="G$1" x="78.74" y="101.6" smashed="yes" rot="R180">
-<attribute name="VALUE" x="80.01" y="109.22" size="1.778" layer="96" rot="R180"/>
-<attribute name="NAME" x="80.01" y="95.758" size="1.778" layer="95" rot="R180"/>
+<instance part="SV1" gate="G$1" x="43.18" y="104.14" smashed="yes" rot="R180">
+<attribute name="VALUE" x="44.45" y="111.76" size="1.778" layer="96" rot="R180"/>
+<attribute name="NAME" x="44.45" y="98.298" size="1.778" layer="95" rot="R180"/>
+</instance>
+<instance part="K1" gate="1" x="71.12" y="93.98" smashed="yes">
+<attribute name="VALUE" x="72.39" y="96.901" size="1.778" layer="96"/>
+<attribute name="PART" x="72.39" y="99.06" size="1.778" layer="95"/>
+</instance>
+<instance part="K1" gate="2" x="17.78" y="101.6" smashed="yes">
+<attribute name="PART" x="20.32" y="101.6" size="1.778" layer="95"/>
+</instance>
+<instance part="K1" gate="3" x="43.18" y="86.36" smashed="yes">
+<attribute name="PART" x="45.72" y="86.36" size="1.778" layer="95"/>
+</instance>
+<instance part="GND5" gate="1" x="71.12" y="86.36" smashed="yes">
+<attribute name="VALUE" x="68.58" y="83.82" size="1.778" layer="96"/>
 </instance>
 </instances>
@@
 </segment>
 <segment>
-<wire x1="20.32" y1="99.06" x2="27.94" y2="99.06" width="0.1524" layer="91"/>
-<pinref part="K2" gate="1" pin="1"/>
-<label x="20.32" y="101.6" size="1.778" layer="95"/>
-<junction x="20.32" y="99.06"/>
-<junction x="27.94" y="99.06"/>
+<wire x1="58.42" y1="99.06" x2="71.12" y2="99.06" width="0.1524" layer="91"/>
+<pinref part="K1" gate="1" pin="+"/>
+<junction x="71.12" y="99.06"/>
+<junction x="58.42" y="99.06"/>
+<label x="58.42" y="101.6" size="1.778" layer="95"/>
 </segment>
 </net>
@@
 </segment>
 <segment>
-<wire x1="43.18" y1="91.44" x2="43.18" y2="93.98" width="0.1524" layer="91"/>
-<pinref part="K2" gate="3" pin="S"/>
-<label x="45.72" y="93.98" size="1.778" layer="95"/>
-<junction x="43.18" y="91.44"/>
-<junction x="43.18" y="93.98"/>
+<wire x1="38.1" y1="91.44" x2="27.94" y2="91.44" width="0.1524" layer="91"/>
+<pinref part="K1" gate="3" pin="S"/>
+<junction x="38.1" y="91.44"/>
+<junction x="27.94" y="91.44"/>
+<label x="27.94" y="93.98" size="1.778" layer="95"/>
 </segment>
 </net>
@@
 </segment>
 <segment>
-<pinref part="K2" gate="1" pin="2"/>
-<pinref part="GND6" gate="1" pin="GND"/>
-<junction x="27.94" y="88.9"/>
+<pinref part="K1" gate="1" pin="-"/>
+<pinref part="GND5" gate="1" pin="GND"/>
+<junction x="71.12" y="88.9"/>
 </segment>
 </net>
@@
 </segment>
 <segment>
-<wire x1="48.26" y1="83.82" x2="55.88" y2="83.82" width="0.1524" layer="91"/>
-<pinref part="K2" gate="3" pin="P"/>
-<label x="58.42" y="83.82" size="1.778" layer="95"/>
-<junction x="48.26" y="83.82"/>
-<junction x="55.88" y="83.82"/>
-</segment>
-</net>
-<net name="N$1" class="0">
-<segment>
-<pinref part="K2" gate="2" pin="P"/>
+<wire x1="43.18" y1="83.82" x2="27.94" y2="83.82" width="0.1524" layer="91"/>
+<pinref part="K1" gate="3" pin="P"/>
+<junction x="43.18" y="83.82"/>
+<junction x="27.94" y="83.82"/>
+<label x="27.94" y="86.36" size="1.778" layer="95"/>
+</segment>
+</net>
+<net name="R-COM" class="0">
+<segment>
+<pinref part="K1" gate="2" pin="P"/>
+<wire x1="17.78" y1="99.06" x2="35.56" y2="99.06" width="0.1524" layer="91"/>
 <pinref part="SV1" gate="G$1" pin="3"/>
-<wire x1="48.26" y1="99.06" x2="71.12" y2="99.06" width="0.1524" layer="91"/>
-<junction x="48.26" y="99.06"/>
-<junction x="71.12" y="99.06"/>
-</segment>
-</net>
-<net name="N$5" class="0">
-<segment>
-<pinref part="K2" gate="2" pin="O"/>
-<wire x1="53.34" y1="106.68" x2="55.88" y2="106.68" width="0.1524" layer="91"/>
-<wire x1="55.88" y1="106.68" x2="55.88" y2="101.6" width="0.1524" layer="91"/>
+<wire x1="35.56" y1="99.06" x2="35.56" y2="101.6" width="0.1524" layer="91"/>
+<junction x="17.78" y="99.06"/>
+<junction x="35.56" y="101.6"/>
+<label x="17.78" y="96.52" size="1.778" layer="95"/>
+</segment>
+</net>
+<net name="R-NC" class="0">
+<segment>
+<pinref part="K1" gate="2" pin="O"/>
+<wire x1="22.86" y1="106.68" x2="22.86" y2="104.14" width="0.1524" layer="91"/>
 <pinref part="SV1" gate="G$1" pin="2"/>
-<wire x1="55.88" y1="101.6" x2="71.12" y2="101.6" width="0.1524" layer="91"/>
-<junction x="53.34" y="106.68"/>
-<junction x="71.12" y="101.6"/>
-</segment>
-</net>
-<net name="N$6" class="0">
-<segment>
+<wire x1="22.86" y1="104.14" x2="35.56" y2="104.14" width="0.1524" layer="91"/>
+<junction x="35.56" y="104.14"/>
+<junction x="22.86" y="106.68"/>
+<label x="25.4" y="104.14" size="1.778" layer="95"/>
+</segment>
+</net>
+<net name="R-NO" class="0">
+<segment>
+<pinref part="K1" gate="2" pin="S"/>
+<wire x1="12.7" y1="106.68" x2="12.7" y2="109.22" width="0.1524" layer="91"/>
+<wire x1="12.7" y1="109.22" x2="35.56" y2="109.22" width="0.1524" layer="91"/>
 <pinref part="SV1" gate="G$1" pin="1"/>
-<wire x1="71.12" y1="104.14" x2="71.12" y2="109.22" width="0.1524" layer="91"/>
-<wire x1="71.12" y1="109.22" x2="43.18" y2="109.22" width="0.1524" layer="91"/>
-<pinref part="K2" gate="2" pin="S"/>
-<wire x1="43.18" y1="109.22" x2="43.18" y2="106.68" width="0.1524" layer="91"/>
-<junction x="43.18" y="106.68"/>
-<junction x="71.12" y="104.14"/>
-</segment>
-</net>
+<wire x1="35.56" y1="109.22" x2="35.56" y2="106.68" width="0.1524" layer="91"/>
+<junction x="12.7" y="106.68"/>
+<junction x="35.56" y="106.68"/>
+<label x="7.62" y="109.22" size="1.778" layer="95"/>
+</segment>
+</net>

Commit message: up
Parts:
- removed X2: P-remote, con-subd:HF26V
- added DCU: DCU, con-lstb:MA08-1
- added J1: 10090926-P264XLF, 10090926-P264XLF:10090926-P264XLF
- added SV2: ANALOG OUT, con-lstb:MA03-1
- added TP1, TP2, TP3, TP4, TP5, TP6, TP7, TP8: TPSQTP13R, testpad:TPSQTP13R
Connections:
- new net AO1: J1.12, SV2.1
- new net D+: DCU.1, J1.24
- new net D-: DCU.2, J1.25
- new net REMOTE_ACTIVE: J1.23, LED3.A, TP5.TP
- net 24+_REMOTE_PRI: now also DCU.7, J1.1, J1.14, TP3.TP; no longer LED3.A, X2.1, X2.14
- net ALARM+: now also J1.19; no longer X2.19
- net ALARM-: now also J1.20; no longer X2.20
- net ERROR: now also J1.9; no longer X2.9
- net GND: now also DCU.8, J1.26, SV2.3, TP1.TP; no longer X2.26
- net NORM+: now also J1.17, TP6.TP; no longer X2.17
- net NORM-: now also J1.16, TP7.TP; no longer X2.16
- net NOT_NORM: now also J1.15, TP8.TP; no longer X2.15
- net SPEED: now also J1.8; no longer X2.8
- net START-: now also J1.3, J1.4, TP2.TP, TP4.TP; no longer X2.3, X2.4
Other:
- moved on the sheet: LED3, R3

Commit message: up
Parts:
- added K2: G6K-2P-Y, relay:G6K-2P-Y
- K1: value G6K-2P -> G6K-2P-Y; device relay:G6K-2P -> relay:G6K-2P-Y
Connections:
- net R-NO renamed N$5
- removed net R-COM: K12.P, SV1.3
- removed net R-NC: K12.O, SV1.2
- new net DECEL_STOP: K12.O, K21.+, SV1.2
- net DECEL+: now also K23.P
- net DECEL-: now also K23.S
- net GND: now also K21.-
- net SPEED: now also K12.P, SV1.3
Other:
- moved on the sheet: SV1
